File: anavi-thermometer-mini.kicad_sch (KiCad schematic)
At the start: 7 parts, among them SW1 SW_DIP_x01, U1 MOUDLE-SEEEDUINO-XIAO-ESP32C6, U2 DS18B20

Commit message: Minor adjustments of the PCB
Signed-off-by: Leon Anavi <leon@anavi.org>
Changed lines of the file:
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@@
+	)
+	(junction
+		(at 177.8 31.75)
+		(diameter 0)
+		(color 0 0 0 0)
+	)
+	(junction
+		(at 177.8 35.56)
+		(diameter 0)
+		(color 0 0 0 0)
 	)
 	(junction
@@
 	(wire
 		(pts
-			(xy 175.26 31.75) (xy 180.34 31.75)
+			(xy 175.26 31.75) (xy 177.8 31.75)
 		)
 		(stroke
@@
 	(wire
 		(pts
-			(xy 175.26 35.56) (xy 179.705 35.56)
+			(xy 175.26 35.56) (xy 177.8 35.56)
 		)
 		(stroke
@@
 	(wire
 		(pts
+			(xy 177.8 35.56) (xy 179.705 35.56)
+		)
+		(stroke
+			(width 0)
+			(type default)
+		)
+	)
+	(wire
+		(pts
 			(xy 228.6 43.815) (xy 228.6 39.37)
 		)
@@
 		(pts
 			(xy 120.65 39.37) (xy 125.73 39.37)
+		)
+		(stroke
+			(width 0)
+			(type default)
+		)
+	)
+	(wire
+		(pts
+			(xy 177.8 31.75) (xy 180.34 31.75)
 		)
 		(stroke
@@
 	)
 	(symbol
+		(lib_id "power:PWR_FLAG")
+		(at 177.8 35.56 180)
+		(unit 1)
+		(exclude_from_sim no)
+		(in_bom yes)
+		(on_board yes)
+		(dnp no)
+		(fields_autoplaced yes)
+		(property "Reference" "#FLG2"
+			(at 177.8 37.465 0)
+			(effects
+				(font
+					(size 1.27 1.27)
+				)
+				(hide yes)
+			)
+		)
+		(property "Value" "PWR_FLAG"
+			(at 177.8 40.64 0)
+			(effects
+				(font
+					(size 1.27 1.27)
+				)
+			)
+		)
+		(property "Footprint" ""
+			(at 177.8 35.56 0)
+			(effects
+				(font
+					(size 1.27 1.27)
+				)
+				(hide yes)
+			)
+		)
+		(property "Datasheet" "~"
+			(at 177.8 35.56 0)
+			(effects
+				(font
+					(size 1.27 1.27)
+				)
+				(hide yes)
+			)
+		)
+		(property "Description" "Special symbol for telling ERC where power comes from"
+			(at 177.8 35.56 0)
+			(effects
+				(font
+					(size 1.27 1.27)
+				)
+				(hide yes)
+			)
+		)
+		(pin "1"
+		)
+		(instances
+			(project ""
+				(path "/2ff006f4-2a61-440d-9643-0ab2f7506f70"
+					(reference "#FLG2")
+					(unit 1)
+				)
+			)
+		)
+	)
+	(symbol
 		(lib_id "Device:R")
 		(at 194.945 46.99 90)
@@
 					(unit 1)
 				)
+			)
+		)
+	)
+	(symbol
+		(lib_id "power:PWR_FLAG")
+		(at 177.8 31.75 0)
+		(unit 1)
+		(exclude_from_sim no)
+		(in_bom yes)
+		(on_board yes)
+		(dnp no)
+		(fields_autoplaced yes)
+		(property "Reference" "#FLG1"
+			(at 177.8 29.845 0)
+			(effects
+				(font
+					(size 1.27 1.27)
+				)
+				(hide yes)
+			)
+		)
+		(property "Value" "PWR_FLAG"
+			(at 177.8 26.67 0)
+			(effects
+				(font
+					(size 1.27 1.27)
+				)
+			)
+		)
+		(property "Footprint" ""
+			(at 177.8 31.75 0)
+			(effects
+				(font
+					(size 1.27 1.27)
+				)
+				(hide yes)
+			)
+		)
+		(property "Datasheet" "~"
+			(at 177.8 31.75 0)
+			(effects
+				(font
+					(size 1.27 1.27)
+				)
+				(hide yes)
+			)
+		)
+		(property "Description" "Special symbol for telling ERC where power comes from"
+			(at 177.8 31.75 0)
+			(effects
+				(font
+					(size 1.27 1.27)
+				)
+				(hide yes)
+			)
+		)
+		(pin "1"
+		)
+		(instances
+			(project ""
+				(path "/2ff006f4-2a61-440d-9643-0ab2f7506f70"
+					(reference "#FLG1")
+					(unit 1)
+				)

Commit message: Use WAGO 2059-303
Replace the three screw terminal block with the more compact
alternative WAGO 2059-303.

Signed-off-by: Leon Anavi <leon@anavi.org>
Parts:
- added D2: LED, LED_SMD:LED_1206_3216Metric, symbol Device:LED
- added R4: 68R, Resistor_SMD:R_0603_1608Metric_Pad0.98x0.95mm_HandSolder, symbol Device:R
- U2: footprint TerminalBlock_Phoenix:TerminalBlock_Phoenix_MKDS-1,5-3_1x03_P5.00mm_Horizontal -> footprints:CONN3_2059-303&slash_998-403_WAG
- renumbered R3 to R1, R1 to R3
Connections:
- net +3V3: now also U2.1 (VDD); no longer U2.3 (VDD)
- net GND: now also U2.5 (GND), D2.1 (K); no longer U2.1 (GND)
- net at R1.1, U1.11 (PA6_A10_D10_MOSI): now also U2.3 (DQ); no longer U2.2 (DQ)
- net at U1.3 (PA10_A2_D2): now also R4.1
- new net: D2.2 (A), R4.2
- no-connect marks 9 -> 8
Other:
- moved on the sheet: D1, R3
